Commit message: Imported upstream version '1.9.0' of 'upstream'

File: tiago_pro_head_description/robots/tiago_pro_head.urdf.xacro (robot description, xacro)
@@ -18,8 +18,10 @@
   <xacro:arg name="is_public_sim" default="false"/>
   <xacro:arg name="namespace" default=""/>
+  <xacro:arg name="gazebo_version" default="classic"/>
   <xacro:property name="camera_model" value="$(arg camera_model)" />
   <xacro:property name="use_sim_time" value="$(arg use_sim_time)" />
   <xacro:property name="is_public_sim" value="$(arg is_public_sim)" />
   <xacro:property name="namespace" value="$(arg namespace)" />
+  <xacro:property name="gazebo_version" value="$(arg gazebo_version)" />
     <!-- ROS 2 Control -->
   <xacro:include filename="$(find tiago_pro_head_description)/ros2_control/ros2_control.urdf.xacro" />

File: tiago_pro_head_description/urdf/head.urdf.xacro (robot description, xacro)
@@ -184,3 +184,9 @@
     <parent link="sellion_link"/>
   </joint>
+  <link name="head_front_camera_color_eye_frame"/>
+  <joint name="color_eye_joint" type="fixed">
+    <origin xyz="0.000 0.000 0.000" rpy="-1.571 0.000 -1.571"/>
+    <child link="head_front_camera_color_eye_frame" />
+    <parent link="head_front_camera_link"/>
+  </joint>
 </robot>

Commit message: Imported upstream version '1.12.0' of 'upstream'

File: tiago_pro_head_description/robots/tiago_pro_head.urdf.xacro (robot description, xacro)
@@ -14,17 +14,36 @@
 <robot xmlns:xacro="http://ros.org/wiki/xacro" name="tiago_pro_head">
   <xacro:include filename="$(find tiago_pro_head_description)/urdf/head.urdf.xacro" />
-  <xacro:arg name="camera_model" default="realsense-d435"/>
+  <xacro:arg name="camera_model" default="realsense-d435i"/>
   <xacro:arg name="use_sim_time" default="false"/>
   <xacro:arg name="is_public_sim" default="false"/>
   <xacro:arg name="namespace" default=""/>
   <xacro:arg name="gazebo_version" default="classic"/>
+  <!-- mujoco-ros2-control, mujoco, gazebo-->
+  <xacro:arg name="sim_type" default="gazebo" />
+  <!-- false, position, motor -->
+  <xacro:arg name="mj_control" default="false" />
+  <!-- floor -->
+  <xacro:arg name="world_name" default="floor" />
   <xacro:property name="camera_model" value="$(arg camera_model)" />
   <xacro:property name="use_sim_time" value="$(arg use_sim_time)" />
   <xacro:property name="is_public_sim" value="$(arg is_public_sim)" />
   <xacro:property name="namespace" value="$(arg namespace)" />
+  <!-- Mujoco properties -->
+  <xacro:property name="sim_type" value="$(arg sim_type)" />
+  <xacro:property name="mj_control" value="$(arg mj_control)"/>
+  <xacro:property name="world_name" value="$(arg world_name)"/>
   <xacro:property name="gazebo_version" value="$(arg gazebo_version)" />
-    <!-- ROS 2 Control -->
-  <xacro:include filename="$(find tiago_pro_head_description)/ros2_control/ros2_control.urdf.xacro" />
-  <xacro:tiago_pro_head_ros2_control/>
+  <!-- Properties check -->
+  <xacro:if value="${sim_type not in ['mujoco-ros2-control', 'mujoco', 'gazebo']}">
+    <xacro:wrong_sim_type />
+  </xacro:if>
+  <xacro:unless value="$(arg use_sim_time)">
+    <xacro:property name="sim_type" value="gazebo" />
+  </xacro:unless>
+  <!-- ROS 2 Control -->
+  <xacro:if value="${sim_type != 'mujoco'}">
+    <xacro:include filename="$(find tiago_pro_head_description)/ros2_control/ros2_control.urdf.xacro" />
+    <xacro:tiago_pro_head_ros2_control use_sim_time="${use_sim_time}" sim_type="${sim_type}"/>
+  </xacro:if>
   <link name="world"/>
   <joint name="head_base_joint" type="fixed">
@@ -65,3 +84,6 @@
   </link>
   <xacro:tiago_pro_head name="head" parent="head_base_link" use_sim_time="$(arg use_sim_time)" camera_model="$(arg camera_model)"/>
+  <xacro:if value="${sim_type in ['mujoco', 'mujoco-ros2-control']}">
+    <xacro:tiago_pro_head_mj world_name="${world_name}" mj_control="${mj_control}"/>
+  </xacro:if>
 </robot>

File: tiago_pro_head_description/ros2_control/ros2_control.urdf.xacro (robot description, xacro)
@@ -13,26 +13,44 @@
  -->
 <robot xmlns:xacro="http://ros.org/wiki/xacro" name="tiago_pro_head" >
-    <xacro:macro name="tiago_pro_head_ros2_control" params="use_sim_time:=^|false">
+  <xacro:macro name="tiago_pro_head_ros2_control" params="use_sim_time:=^|false sim_type:=^|gazebo">
     <xacro:include filename="$(find tiago_pro_head_description)/urdf/head.ros2_control.xacro" />
-    <xacro:unless value="$(arg use_sim_time)">
-      <ros2_control name="ros2_control_tiago_pro_head_system" type="system">
+    <ros2_control name="ros2_control_tiago_pro_head_system" type="system">
         <hardware>
-          <plugin>robot_control/RobotControl</plugin>
+          <xacro:if value="${use_sim_time}">
+            <xacro:if value="${sim_type == 'gazebo'}">
+              <xacro:if value="${gazebo_version == 'classic'}">
+                <plugin>gazebo_ros2_control/GazeboSystem</plugin>
+              </xacro:if>
+              <xacro:if value="${gazebo_version == 'gazebo'}">
+                <plugin>gz_ros2_control/GazeboSimSystem</plugin>
+              </xacro:if>
+            </xacro:if>
+            <xacro:if value="${sim_type == 'mujoco-ros2-control'}">
+              <plugin>mujoco_ros2_control/MujocoSystemInterface</plugin>
+              <!-- Override the slowdown settings in the Simulate App and run at 3x speed -->
+              <param name="sim_speed_factor">1.0</param>
+            </xacro:if>
+          </xacro:if>
+          <xacro:unless value="${use_sim_time}">
+            <plugin>robot_control/RobotControl</plugin>
+          </xacro:unless>
         </hardware>
-        <xacro:ros2_control_head />
-      </ros2_control>
-    </xacro:unless>
-    <xacro:if value="$(arg use_sim_time)">
-      <gazebo>
-        <plugin filename="libgazebo_ros2_control.so" name="gazebo_ros2_control">
-          <parameters>$(find tiago_pro_head_description)/ros2_control/gazebo_controller_manager_cfg.yaml</parameters>
-        </plugin>
-      </gazebo>
-      <ros2_control name="ros2_control_head_gazebo_system" type="system">
-        <hardware>
-          <plugin>gazebo_ros2_control/GazeboSystem</plugin>
-        </hardware>
-        <xacro:ros2_control_head />
-      </ros2_control>
+        <xacro:ros2_control_head sim_type="${sim_type}"/>
+    </ros2_control>
+    <xacro:if value="${use_sim_time}">
+      <xacro:if value="${sim_type == 'gazebo'}">
+        <xacro:if value="${gazebo_version == 'classic'}">
+          <plugin filename="libgazebo_ros2_control.so" name="gazebo_ros2_control">
+            <parameters>$(find tiago_pro_head_description)/ros2_control/gazebo_controller_manager_cfg.yaml</parameters>
+          </plugin>
+        </xacro:if>
+        <xacro:if value="${gazebo_version == 'gazebo'}">
+          <plugin filename="gz_ros2_control-system" name="gz_ros2_control::GazeboSimROS2ControlPlugin">
+            <robot_param>robot_description</robot_param>
+            <robot_param_node>robot_state_publisher</robot_param_node>
+            <parameters>$(find tiago_pro_head_description)/ros2_control/gazebo_controller_manager_cfg.yaml</parameters>
+          </plugin>
+        </xacro:if>
+      </xacro:if>
     </xacro:if>
   </xacro:macro>

File: tiago_pro_head_description/urdf/head.ros2_control.xacro (robot description, xacro)
@@ -14,9 +14,9 @@
 <robot xmlns:xacro="http://ros.org/wiki/xacro">
   <!-- ROS 2 Control -->
-  <xacro:macro name="ros2_control_head" >
-    <xacro:ros2_control_head_joint name="head_1" reduction="1.0" offset_value="0.0" />
-    <xacro:ros2_control_head_joint name="head_2" reduction="1.0" offset_value="0.0" />
+  <xacro:macro name="ros2_control_head" params="sim_type:=^|gazebo">
+    <xacro:ros2_control_head_joint name="head_1" reduction="1.0" offset_value="0.0" sim_type="${sim_type}" />
+    <xacro:ros2_control_head_joint name="head_2" reduction="1.0" offset_value="0.0" sim_type="${sim_type}"/>
   </xacro:macro>
-  <xacro:macro name="ros2_control_head_joint" params="name reduction offset_value" >
+  <xacro:macro name="ros2_control_head_joint" params="name reduction offset_value sim_type:=^|gazebo" >
     <joint name="${name}_joint">
       <command_interface name="position" />
@@ -26,5 +26,5 @@
     </joint>
     <xacro:include filename="$(find tiago_pro_head_description)/urdf/head.transmission.urdf.xacro" />
-    <xacro:head_transmission name="${name}" reduction="1" offset_value="${offset_value}" />
+    <xacro:head_transmission name="${name}" reduction="1" offset_value="${offset_value}" sim_type="${sim_type}"/>
   </xacro:macro>
 </robot>

File: tiago_pro_head_description/urdf/head.transmission.urdf.xacro (robot description, xacro)
@@ -13,11 +13,16 @@
 -->
 <robot xmlns:xacro="http://ros.org/wiki/xacro">
-  <xacro:macro name="head_transmission" params="name reduction offset_value">
+  <xacro:macro name="head_transmission" params="name reduction offset_value sim_type:=^gazebo">
     <transmission name="${name}_trans">
       <plugin>transmission_interface/SimpleTransmission</plugin>
-      <actuator name="${name}_actuator" role="actuator1"/>
+      <xacro:if value="${sim_type == 'mujoco-ros2-control'}">
+        <actuator name="${name}_joint" role="actuator1"/>
+      </xacro:if>
+      <xacro:unless value="${sim_type == 'mujoco-ros2-control'}">
+        <actuator name="${name}_actuator" role="actuator1"/>
+      </xacro:unless>
       <joint name="${name}_joint" role="joint1" >
         <offset>${offset_value}</offset>
-        <mechanicalReduction>${reduction}</mechanicalReduction>
+        <mechanical_reduction>${reduction}</mechanical_reduction>
       </joint>
     </transmission>

File: tiago_pro_head_description/urdf/head.urdf.xacro (robot description, xacro)
@@ -13,19 +13,13 @@
 -->
 <robot xmlns:xacro="http://ros.org/wiki/xacro">
-  <!--File includes-->
-  <xacro:include filename="$(find pal_urdf_utils)/urdf/camera/realsense_d435.urdf.xacro" />
-  <xacro:include filename="$(find pal_urdf_utils)/urdf/camera/realsense_d455.urdf.xacro" />
-  <!-- Tools -->
-  <xacro:include filename="$(find pal_urdf_utils)/urdf/deg_to_rad.urdf.xacro" />
-  <!--Constant parameters-->
-  <xacro:property name="head_friction" value="1.0" />
-  <xacro:property name="head_damping" value="0.5" />
-  <xacro:property name="head_max_vel" value="3.0" />
-  <xacro:property name="head_1_lower_limit" value="-1.309"/>
-  <xacro:property name="head_1_upper_limit" value="1.309"/>
-  <xacro:property name="head_2_lower_limit" value="-1.0472"/>
-  <xacro:property name="head_2_upper_limit" value="0.34907"/>
-  <xacro:property name="head_eps" value="${0.07}" />
   <xacro:macro name="tiago_pro_head" params="name parent camera_model use_sim_time:=^|false">
+    <!--File includes-->
+    <xacro:include filename="$(find pal_urdf_utils)/urdf/camera/realsense_d435.urdf.xacro" />
+    <xacro:include filename="$(find pal_urdf_utils)/urdf/camera/realsense_d435i.urdf.xacro" />
+    <xacro:include filename="$(find pal_urdf_utils)/urdf/camera/realsense_d455.urdf.xacro" />
+     <!-- Tools -->
+    <xacro:property name="head_eps" value="${0.07}" />
+    <xacro:include filename="$(find pal_urdf_utils)/urdf/deg_to_rad.urdf.xacro" />
+    <xacro:include filename="$(find tiago_pro_head_description)/urdf/head_limits.xacro" />
     <!-- Head Link 1-->
     <link name="${name}_1_link">
@@ -58,5 +52,5 @@
       <child link="head_1_link" />
       <axis xyz="0 0 1" />
-      <limit lower="${head_1_lower_limit}" upper="${head_1_upper_limit}" effort="5.197" velocity="${head_max_vel}" />
+      <limit lower="${head_1_lower_limit}" upper="${head_1_upper_limit}" effort="${head_1_max_effort}" velocity="${head_max_vel}" />
       <dynamics damping="${head_damping}" friction="${head_friction}"/>
       <safety_controller k_position="20" k_velocity="20" soft_lower_limit="${head_1_lower_limit + head_eps}" soft_upper_limit="${head_1_upper_limit - head_eps}" />
@@ -101,5 +95,5 @@
       <child link="${name}_2_link" />
       <axis xyz="0 0 -1" />
-      <limit lower="${head_2_lower_limit}" upper="${head_2_upper_limit}" effort="2.77" velocity="${head_max_vel}" />
+      <limit lower="${head_2_lower_limit}" upper="${head_2_upper_limit}" effort="${head_2_max_effort}" velocity="${head_max_vel}" />
       <dynamics damping="${head_damping}" friction="${head_friction}"/>
       <safety_controller k_position="20" k_velocity="20" soft_lower_limit="${head_2_lower_limit + head_eps}" soft_upper_limit="${head_2_upper_limit - head_eps}" />
@@ -116,18 +110,20 @@
       </visual>
     </link>
-    <gazebo reference="${name}_screen_link">
-      <visual>
-        <plugin name="${name}_video_stream" filename="libgazebo_ros_video.so">
-          <ros>
-            <!-- Add a namespace -->
-            <namespace></namespace>
-            <!-- remap image subscribe topic -->
-            <remapping>~/image_raw:=robot_face/image_raw</remapping>
-          </ros>
-          <height>480</height>
-          <width>640</width>
-        </plugin>
-      </visual>
-    </gazebo>
+    <xacro:if value="${gazebo_version == 'classic'}">
+      <gazebo reference="${name}_screen_link">
+        <visual>
+          <plugin name="${name}_video_stream" filename="libgazebo_ros_video.so">
+            <ros>
+              <!-- Add a namespace -->
+              <namespace></namespace>
+              <!-- remap image subscribe topic -->
+              <remapping>~/image_raw:=robot_face/image_raw</remapping>
+            </ros>
+            <height>480</height>
+            <width>640</width>
+          </plugin>
+        </visual>
+      </gazebo>
+    </xacro:if>
     <joint name="${name}_screen_joint" type="fixed">
       <parent link="${name}_2_link" />
@@ -152,4 +148,10 @@
     </gazebo>
     <!-- Cameras-->
+    <!-- Head camera:Intel D435i -->
+    <xacro:if value="${camera_model == 'realsense-d435i'}">
+      <xacro:realsense_d435i parent="${name}_2_link" name="${name}_front_camera" use_nominal_extrinsics="${use_sim_time}">
+        <origin xyz="0.0416 -0.1555 0" rpy="1.5708 0 0" />
+      </xacro:realsense_d435i>
+    </xacro:if>
     <!-- Head camera:Intel D435 -->
     <xacro:if value="${camera_model == 'realsense-d435'}">
@@ -164,4 +166,46 @@
       </xacro:realsense_d455>
     </xacro:if>
+  </xacro:macro>
+  <xacro:macro name="tiago_pro_head_mj" params="mj_control world_name">
+    <xacro:include filename="$(find tiago_pro_head_description)/mujoco/mj_tags.xacro" />
+    <xacro:include filename="$(find pal_mujoco_scenes)/scenes/${world_name}.xacro" />
+    <mujoco_inputs>
+      <!-- Mujoco environment -->
+      <scene>
+        <xacro:mj_scene/>
+      </scene>
+      <raw_inputs>
+        <!-- Actuator-->
+        <actuator>
+          <xacro:mj_head_actuators mj_control="${mj_control}"/>
+        </actuator>
+        <default>
+          <default class="visual">
+            <geom group="2" type="mesh" contype="0" conaffinity="0"/>
+          </default>
+          <default class="collision">
+            <geom group="3" type="mesh"/>
+          </default>
+        </default>
+      </raw_inputs>
+      <processed_inputs>
+        <!-- Specifying decompose_mesh will set the `decompose` flag when using obj2mjcf -->
+        <!-- <decompose_mesh mesh_name="{mesh_name}" threshold=" {threshold_value}"/> -->
+        <!-- The camera with the specified values will be added at the specified site name. -->
+        <!-- The position and quaterinion will be filled in by the converter -->
+        <!-- Realsense_d435 -->
+        <!-- <camera site="head_front_camera_color_eye_frame" name="head" fovy="42" mode="fixed" resolution="848 480"/> -->
+        <!-- Adds a lidar tag below a site tag to support a lidar sensor. -->
+        <!-- In the URDF, we assume that that the sensor frame has the Z-axis pointed directly up in the sensor -->
+        <!-- frame. This tag will create rangefinders in the MJCF between min_angle and max_angle at each -->
+        <!-- angle_increment rotated about the replicate frame's Y axis. The hardware intercface then combines -->
+        <!-- them into a single LaserScan message. -->
+        <!-- <lidar ref_site="{link_name}" sensor_name="{sensor_name}" min_angle="{min_angle_value}" max_angle="{max_angle_value}" angle_increment="{angle_increment_value}" /> -->
+        <!-- The element with the type and name as listed below will be modified with the remaining attributes -->
+        <!-- If the attribute already existed, it will be overwritten -->
+        <!-- Note that the type and name elements are required -->
+        <!-- <modify_element type="{element_type}" name="{element_name}" frictionloss="{value}" damping="{value}"/> -->
+      </processed_inputs>
+    </mujoco_inputs>
   </xacro:macro>
   <!-- EYE FRAMES -->
